File: MicroCerveceria.kicad_sch (KiCad schematic)
At the start: 5 parts, among them J1 BORNERA-2

Commit message: Finaliza PCB
Other:
- sheet core ports: added GPIO10, GPIO12, GPIO9; removed none
- sheet entradas ports: added ENTRADA_onewire_OUT; removed none
- sheet salidas ports: added RELE_3_IN, RELE_4_IN; removed none
