File: entradas.kicad_sch (KiCad schematic)
At the start: 14 parts, among them J5 BORNERA-2, J6 BORNERA-2, J9 Screw_Terminal_01x03, U4 TLP621, U5 TLP621

Commit message: Finaliza PCB
Connections:
- net ENTRADA_1_OUT: now also R10.2, U5.4; no longer R8.2, U4.4
- net ENTRADA_2_OUT: now also R8.2, U4.4; no longer R10.2, U5.4
