File: salidas.kicad_sch (KiCad schematic)
At the start: 28 parts, among them J3 BORNERA-3, J4 BORNERA-3, J7 BORNERA-3, J8 BORNERA-3, K1 SANYOU_SRD_Form_C, K2 SANYOU_SRD_Form_C, K3 SANYOU_SRD_Form_C, K4 SANYOU_SRD_Form_C, Q1 2N7002K, Q2 2N7002K, Q3 2N7002K, Q4 2N7002K

Commit message: Finaliza PCB
Connections:
- net RELE_1_IN: no longer Q3.1 (G), R17.1
- net RELE_2_IN: no longer Q4.1 (G), R19.1
- net at J4.2 (Pin_2): now also K2.3; no longer K2.4
- net at J4.3 (Pin_3): now also K2.4; no longer K2.3
- net at J7.1 (Pin_1): now also K3.1; no longer K3.4
- net at J7.3 (Pin_3): now also K3.4; no longer K3.1
- net at J3.1 (Pin_1): now also K1.1; no longer K1.4
- net at J3.3 (Pin_3): now also K1.4; no longer K1.1
- net at J8.2 (Pin_2): now also K4.3; no longer K4.4
- net at J8.3 (Pin_3): now also K4.4; no longer K4.3
- new net RELE_3_IN: Q3.1 (G), R17.1
- new net RELE_4_IN: Q4.1 (G), R19.1
Other:
- moved on the sheet: J3, J7
