File: MicroCerveceria.kicad_pcb (KiCad board)
At the start: 2 copper layers, 73 parts, among them J1 BORNERA-2, J2 PINM-6, J3 BORNERA-3, J4 BORNERA-3, J5 BORNERA-2, J6 BORNERA-2, J7 BORNERA-3, J8 BORNERA-3, J9 Screw_Terminal_01x03, K1 SANYOU_SRD_Form_C, K2 SANYOU_SRD_Form_C, K3 SANYOU_SRD_Form_C, K4 SANYOU_SRD_Form_C, Q1 2N7002K, Q2 2N7002K, Q3 2N7002K, Q4 2N7002K, SW1 TACT-SWITCH 7 mm, U1 LM2596S-ADJ, U2 LM1117-3.3, U3 ESP-12F, U4 TLP621, U5 TLP621

Commit message: Finaliza PCB
Parts:
- moved D7 244.0 mm to (22.7, 89.8), turned to 180 degrees
- moved R12 227.7 mm to (27.6, 89.8), turned to 180 degrees
- moved R6 213.5 mm to (48.0, 83.2), turned to 90 degrees
- moved Q1 212.4 mm to (43.5, 83.1), turned to 180 degrees
- moved R13 206.7 mm to (27.6, 93.5), turned to 180 degrees
- moved D8 204.9 mm to (22.7, 93.5), turned to 180 degrees
- moved D3 202.9 mm to (35.6, 83.1)
- moved R7 186.7 mm to (67.6, 83.2), turned to 90 degrees
- moved D12 184.6 mm to (74.4, 83.1)
- moved J3 179.1 mm to (35.5, 113.1)
- moved J7 177.1 mm to (73.1, 113.1)
- moved D4 174.5 mm to (55.6, 83.1)
- moved Q4 167.2 mm to (101.6, 83.1), turned to 180 degrees
- moved D14 166.8 mm to (93.7, 83.1)
- moved R19 165.2 mm to (106.7, 83.2), turned to 90 degrees
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Connections:
- J3 pad 1: Net-(J3-Pad1) -> Net-(J3-Pin_1)
- J3 pad 3: Net-(J3-Pad3) -> Net-(J3-Pin_3)
- J4 pad 2: Net-(J4-Pad2) -> Net-(J4-Pin_2)
- J4 pad 3: Net-(J4-Pad3) -> Net-(J4-Pin_3)
- J7 pad 1: Net-(J7-Pad1) -> Net-(J7-Pin_1)
- J7 pad 3: Net-(J7-Pad3) -> Net-(J7-Pin_3)
- J8 pad 2: Net-(J8-Pad2) -> Net-(J8-Pin_2)
- J8 pad 3: Net-(J8-Pad3) -> Net-(J8-Pin_3)
- J9 pad 2: /GPIO12 -> /core/GPIO12
- K1 pad 1: Net-(J3-Pad3) -> Net-(J3-Pin_1)
- K1 pad 4: Net-(J3-Pad1) -> Net-(J3-Pin_3)
- K2 pad 3: Net-(J4-Pad3) -> Net-(J4-Pin_2)
- K2 pad 4: Net-(J4-Pad2) -> Net-(J4-Pin_3)
- K3 pad 1: Net-(J7-Pad3) -> Net-(J7-Pin_1)
- K3 pad 4: Net-(J7-Pad1) -> Net-(J7-Pin_3)
- K4 pad 3: Net-(J8-Pad3) -> Net-(J8-Pin_2)
- K4 pad 4: Net-(J8-Pad2) -> Net-(J8-Pin_3)
- Q1 pad 1: /core/GPIO5 -> /core/GPIO9
- Q2 pad 1: /core/GPIO4 -> /core/GPIO10
- Q3 pad 1: /GPIO9 -> /core/GPIO4
- Q4 pad 1: /GPIO10 -> /core/GPIO5
- R10 pad 2: /core/GPIO13 -> /core/GPIO14
- R17 pad 1: /GPIO9 -> /core/GPIO4
- R19 pad 1: /GPIO10 -> /core/GPIO5
- R20 pad 2: /GPIO12 -> /core/GPIO12
- R6 pad 1: /core/GPIO5 -> /core/GPIO9
- R7 pad 1: /core/GPIO4 -> /core/GPIO10
- R8 pad 2: /core/GPIO14 -> /core/GPIO13
- U4 pad 4: /core/GPIO14 -> /core/GPIO13
- U5 pad 4: /core/GPIO13 -> /core/GPIO14
Routing:
- net GND: track 142.0 -> 456.1 mm, vias 2 -> 38
- net +5V: track 47.7 -> 254.4 mm, vias 0 -> 5
- net +3V3: track 22.5 -> 174.7 mm, vias 0 -> 4
- net /core/GPIO9: track 0.00 -> 73.7 mm
- net +VSW: track 30.5 -> 96.7 mm
- net Net-(J2-Pin_2): track 0.00 -> 56.0 mm, vias 0 -> 2
- net /core/GPIO10: track 0.00 -> 54.6 mm
- net Net-(D12-A): track 0.00 -> 54.3 mm, vias 0 -> 2
- net Net-(D4-A): track 0.00 -> 52.7 mm
- net /core/GPIO14: track 0.00 -> 48.3 mm, vias 0 -> 1
- net /core/GPIO13: track 0.00 -> 41.4 mm, vias 0 -> 1
- net /core/GPIO4: track 0.00 -> 41.3 mm, vias 0 -> 2
- net /core/GPIO12: track 0.00 -> 40.0 mm, vias 0 -> 1
- net Net-(J7-Pin_1): track 0.00 -> 37.2 mm
- net Net-(J4-Pin_1): track 0.00 -> 36.8 mm
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- added copper zone on B.Cu, net GND
- added copper zone on F.Cu, net GND
Other:
- board outline added: 100 x 100 mm
- board text added: "Micro-Monitor v. _ . _ 4S2E1WIRE"

Commit message: Creacion gerber y listado de componentes
Routing:
- net Net-(J4-Pin_1): track 36.8 -> 37.8 mm
